File: experiments/30-flight-computer-pcb/hardware/kicad/cc-flight-logger.kicad_pcb (KiCad board)
At the start: 2 copper layers, 80 x 30 mm, 47 parts, among them J1 USB-C (power only), J2 LiPo 1S, J3 PWR SW, J4 microSD, J5 RADIO (RFM95W), J6 GPS UART, J7 EXT BEEPER, Q1 MMBT3904, U1 Raspberry Pi Pico, U2 MCP73831-2-OT, U3 LSM6DSO32, U4 BMP390, U5 AP2112K-3.3

Commit message: Rename to Cosmic Library; add booster, Moon and Mars landings, rocket hangar, live Earth orbit, night sky, cosmic scale
Other:
- board text added: "cosmic-library CC-FL1"
- board text removed: "cosmic-codex CC-FL1"
Changed lines of the file:
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@@
   (gr_line (start 178.5 130) (end 101.5 130)
     (stroke (width 0.1) (type default)) (layer "Edge.Cuts"))
-  (gr_text "cosmic-codex  CC-FL1" (at 120 128.9) (layer "B.SilkS")
+  (gr_text "cosmic-library  CC-FL1" (at 120 128.9) (layer "B.SilkS")
     (effects (font (size 0.8 0.8) (thickness 0.12)) (justify mirror))
   )
