File: experiments/30-flight-computer-pcb/hardware/kicad/cc-flight-logger.kicad_sch (KiCad schematic)
At the start: 47 parts, among them J1 USB-C (power only), J2 LiPo 1S, J3 PWR SW, J4 microSD, J5 RADIO (RFM95W), J6 GPS UART, J7 EXT BEEPER, Q1 MMBT3904, U1 Raspberry Pi Pico, U2 MCP73831-2-OT, U3 LSM6DSO32, U4 BMP390, U5 AP2112K-3.3

Commit message: Rename to Cosmic Library; add booster, Moon and Mars landings, rocket hangar, live Earth orbit, night sky, cosmic scale
Other:
- company: Cosmic Codex - github.com/Normansrule/cosmic-codex -> Cosmic Library - github.com/Normansrule/cosmic-library
- title: Cosmic Codex Flight Logger CC-FL1 -> Cosmic Library Flight Logger CC-FL1
Changed lines of the file:
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@@
   (paper "A3")
   (title_block
-    (title "Cosmic Codex Flight Logger CC-FL1")
+    (title "Cosmic Library Flight Logger CC-FL1")
     (date "2026-09-26")
     (rev "A")
-    (company "Cosmic Codex - github.com/Normansrule/cosmic-codex")
+    (company "Cosmic Library - github.com/Normansrule/cosmic-library")
     (comment 1 "Rocket flight DATA LOGGER: barometer + IMU + microSD + beeper + telemetry header")
     (comment 2 "Generated by hardware/scripts/generate.py from design.py - edit design.py, not this file")
